File: Hardware 1.4 (By Popopo)/MDP_Cartridge_Large/MicroPicoDriveCartridge.kicad_sch (KiCad schematic)
At the start: 11 parts, among them J1 Conn_02x08_Odd_Even, SW1 SW_Push, SW2 SW_Push, SW3 SW_Push

Commit message: recovering hard format
Connections:
- net GND: now also J1.16 (Pin_16)
- no-connect marks 5 -> 4
Other:
- note added: "Pin#14 > Signal UI_DETECT. Takes UI_DETECT signal to GND to indicate the cartridge is inserted."
- note removed: "Pin#14 > Signal UI_DETECT. Recive UI_DETECT signal in order to indicate the cartridge is inserted."
Changed lines of the file:
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@@
 		)
 	)
-	(text "Pin#14 > Signal UI_DETECT.\nRecive UI_DETECT signal in order to indicate the cartridge is inserted."
+	(text "Pin#14 > Signal UI_DETECT.\nTakes UI_DETECT signal to GND to indicate the cartridge is inserted."
 		(exclude_from_sim no)
 		(at 170.18 106.68 0)
@@
 			(justify left bottom)
 		)
+	)
+	(junction
+		(at 213.36 101.6)
+		(diameter 0)
+		(color 0 0 0 0)
 	)
 	(junction
@@
 	)
 	(no_connect
-		(at 212.09 101.6)
-	)
-	(no_connect
 		(at 185.42 134.62)
 	)
@@
 	(wire
 		(pts
+			(xy 213.36 99.06) (xy 213.36 101.6)
+		)
+		(stroke
+			(width 0)
+			(type default)
+		)
+	)
+	(wire
+		(pts
 			(xy 87.63 87.63) (xy 86.36 87.63)
 		)
@@
 	(wire
 		(pts
+			(xy 212.09 99.06) (xy 213.36 99.06)
+		)
+		(stroke
+			(width 0)
+			(type default)
+		)
+	)
+	(wire
+		(pts
 			(xy 99.06 91.44) (xy 99.06 95.25)
 		)
@@
 	(wire
 		(pts
+			(xy 213.36 101.6) (xy 217.17 101.6)
+		)
+		(stroke
+			(width 0)
+			(type default)
+		)
+	)
+	(wire
+		(pts
 			(xy 212.09 86.36) (xy 214.63 86.36)
 		)
@@
 	(wire
 		(pts
-			(xy 212.09 99.06) (xy 213.36 99.06)
+			(xy 212.09 101.6) (xy 213.36 101.6)
 		)
 		(stroke
@@
 	(symbol
 		(lib_id "power:GND")
-		(at 213.36 99.06 90)
+		(at 217.17 101.6 90)
 		(mirror x)
 		(unit 1)
@@
 		(dnp no)
 		(property "Reference" "#PWR03"
-			(at 219.71 99.06 0)
+			(at 223.52 101.6 0)
 			(effects
 				(font
@@
 		)
 		(property "Value" "GND"
-			(at 220.98 99.06 90)
+			(at 224.79 101.6 90)
 			(effects
 				(font
@@
 		)
 		(property "Footprint" ""
-			(at 213.36 99.06 0)
+			(at 217.17 101.6 0)
 			(effects
 				(font
@@
 		)
 		(property "Datasheet" ""
-			(at 213.36 99.06 0)
+			(at 217.17 101.6 0)
 			(effects
 				(font
@@
 		)
 		(property "Description" "Power symbol creates a global label with name \"GND\" , ground"
-			(at 213.36 99.06 0)
-			(effects
-				(font
+			(at 217.17 101.6 0)
+			(effects
+				(font
