File: Hardware 1.4 (By Popopo)/MDP_Cartridge_Large/MicroPicoDriveCartridge.kicad_pcb (KiCad board)
At the start: 2 copper layers, 37.2 x 37.5 mm, 11 parts, among them J1 Conn_02x08_Odd_Even, SW1 SW_Push, SW2 SW_Push, SW3 SW_Push

Commit message: recovering hard format
Connections:
- J1 pad 16: unconnected-(J1-Pin_16-Pad16) -> GND
Routing:
- net GND: track 14.8 -> 21.7 mm, vias 12 -> 15
Other:
- board size 37.2 x 37.5 mm -> 37.9 x 37.5 mm
- board text added: "Pin#14 is UI_Detect that close the grund laze when the cartridge is inserted."

Commit message: changing DRC and PCB references 2
Routing:
- net GND: track 21.7 -> 22.9 mm, vias 15 -> 19
- net /UI_BTN_BACK: track 48.4 -> 49.5 mm
