File: Hardware 1.4 (By Popopo)/MDP_Cartridge_Large/MicroPicoDriveCartridge.kicad_pcb (KiCad board)
At the start: 2 copper layers, 37.9 x 37.5 mm, 11 parts, among them J1 Conn_02x08_Odd_Even, SW1 SW_Push, SW2 SW_Push, SW3 SW_Push

Commit message: last changes
Other:
- board text added: "WayWayWay"
Changed lines of the file:
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@@
+		)
+	)
+	(gr_text "WayWayWay"
+		(at 141.7 107.2 0)
+		(layer "B.SilkS")
+		(effects
+			(font
+				(size 1 1)
+				(thickness 0.15)
+			)
+			(justify left bottom mirror)
 		)
 	)

Commit message: deep revision hardw & github info
Routing:
- net GND: vias 19 -> 20
Other:
- board size 37.9 x 37.5 mm -> 30.8 x 36 mm
- board text added: "Redesigned by Popopo (2026) Original design by Dr. Gusman"
- board text removed: "2023 Redesigned by Popopo Original design by Dr. Gusman"
Changed lines of the file:
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@@
 		(sheetfile "MicroPicoDriveCartridge.kicad_sch")
 		(attr allow_missing_courtyard)
+		(fp_rect
+			(start -11.7 -4.95)
+			(end 11.75 3.3)
+			(stroke
+				(width 0.1)
+				(type solid)
+			)
+			(fill yes)
+			(layer "F.Mask")
+		)
+		(fp_rect
+			(start -11.5 -4.95)
+			(end 11.55 3.3)
+			(stroke
+				(width 0.1)
+				(type solid)
+			)
+			(fill yes)
+			(layer "B.Mask")
+		)
 		(fp_line
-			(start -15.4 5.4)
+			(start -15.4 31.63)
 			(end -15.4 -2.590983)
 			(stroke
@@
 		)
 		(fp_line
-			(start 15.4 5.4)
+			(start 15.4 31.63)
 			(end 15.4 -2.590983)
 			(stroke
@@
 		)
 		(pad "14" smd roundrect
-			(at 6.35 1.25)
-			(size 2 5.5)
+			(at 6.35 1.5)
+			(size 2 5)
 			(layers "B.Cu" "B.Mask" "B.Paste")
 			(roundrect_rratio 0.25)
@@
 		)
 	)
-	(gr_rect
-		(start 130.93 63.17)
-		(end 154.85 71.18)
-		(stroke
-			(width 0.15)
-			(type solid)
-		)
-		(fill yes)
-		(layer "F.Mask")
-	)
-	(gr_rect
-		(start 130.93 63.17)
-		(end 154.85 71.18)
-		(stroke
-			(width 0.15)
-			(type solid)
-		)
-		(fill yes)
-		(layer "B.Mask")
-	)
 	(gr_arc
 		(start 127.02094 110.886682)
@@
 	)
 	(gr_line
-		(start 127.31 73.37)
-		(end 127.345938 99.510524)
-		(stroke
-			(width 0.1)
-			(type solid)
-		)
-		(layer "Edge.Cuts")
-	)
-	(gr_line
-		(start 127.345938 99.510524)
+		(start 127.31 99.6)
 		(end 124.254061 106.089475)
 		(stroke
@@
 	)
 	(gr_line
-		(start 158.11 73.37)
-		(end 158.125 99.523873)
+		(start 158.11 99.6)
+		(end 161.322348 106.047317)
 		(stroke
 			(width 0.1)
@@
 	)
 	(gr_line
-		(start 158.125 99.523873)
-		(end 161.216877 106.102824)
+		(start 158.450059 110.900031)
+		(end 127.020922 110.886682)
 		(stroke
 			(width 0.1)
@@
 		(layer "Edge.Cuts")
 	)
-	(gr_line
-		(start 158.450059 110.900031)
-		(end 127.020922 110.886682)
+	(gr_arc
+		(start 161.322348 106.045313)
+		(mid 161.751038 107.615398)
+		(end 161.33965 109.190105)
 		(stroke
 			(width 0.1)
@@
 	)
 	(gr_arc
-		(start 161.216876 106.102824)
-		(mid 161.258209 109.323191)
-		(end 158.449998 110.900031)
+		(start 161.330763 109.190105)
+		(mid 160.136271 110.459267)
+		(end 158.450059 110.900031)
 		(stroke
 			(width 0.1)
@@
 		)
 	)
-	(gr_text "2023 Redesigned by Popopo\nOriginal design by Dr. Gusman"
+	(gr_text "Redesigned by Popopo (2026)\nOriginal design by Dr. Gusman"
 		(at 157.65 74.55 90)
 		(layer "B.SilkS")
@@
 	)
 	(via
-		(at 133.05 88.3)
+		(at 132.05 89.75)
 		(size 0.8)
 		(drill 0.4)
@@
 	)
 	(via
+		(at 147.5 86.7)
+		(size 0.8)
+		(drill 0.4)
+		(layers "F.Cu" "B.Cu")
+		(free yes)
+		(net 1)
+	)
+	(via
 		(at 132.375 103.675)
 		(size 0.8)
@@
 	)
 	(via
-		(at 140.9 88)
+		(at 141 87.85)
 		(size 0.8)
 		(drill 0.4)
