File: Hardware 1.4 (By Popopo)/MDP_Cartridge_Short/MicroPicoDriveCartridge.kicad_pcb (KiCad board)
At the start: 2 copper layers, 33.9 x 37.6 mm, 11 parts, among them J1 Conn_02x08_Odd_Even, SW1 SW_Push, SW2 SW_Push, SW3 SW_Push

Commit message: recovering hard format
Parts:
- moved C1 0.20 mm to (138.0, 90.2)
Connections:
- J1 pad 16: unconnected-(J1-Pin_16-Pad16) -> GND
Routing:
- net GND: track 14.8 -> 22.8 mm, vias 12 -> 15
Other:
- board size 33.9 x 37.6 mm -> 33.9 x 37.5 mm
- board text added: "2023 Redesigned by Popopo Original design by Dr. Gusman"
- board text added: "Important. The mSD limit is place to the EDGE of the cartridge, if any of those vary it could not fit the perfect place that is set now."
- board text added: "Pin#14 is UI_Detect that close the grund laze when the cartridge is inserted."
- board text added: "Ver 1.4e.L"
- board text removed: "2024 Redesigned by Popopo Original design by Dr. Gusman"
- board text removed: "Ver 1.4.eS"
