File: Hardware 1.4 (By Popopo)/MDP_Cartridge_Short/MicroPicoDriveCartridge.kicad_pcb (KiCad board)
At the start: 2 copper layers, 33.9 x 37.5 mm, 11 parts, among them J1 Conn_02x08_Odd_Even, SW1 SW_Push, SW2 SW_Push, SW3 SW_Push

Commit message: Last changes on dev PCBs
Other:
- board text added: "Pin#14 is UI_Detect that close the ground laze when the cartridge is inserted."
- board text removed: "Pin#14 is UI_Detect that close the grund laze when the cartridge is inserted."
Changed lines of the file:
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@@
 	)
 	(gr_text "Important.\nThe mSD limit is place to the EDGE of the cartridge, \nif any of those vary it could not fit the perfect place that is set now."
-		(at 148.1 118.5 0)
+		(at 150.49 126.59 0)
 		(layer "Cmts.User")
 		(effects
@@
 		)
 	)
-	(gr_text "Pin#14 is UI_Detect that close the grund laze when the cartridge is inserted."
-		(at 171.725 68.6 0)
+	(gr_text "Pin#14 is UI_Detect that close the ground laze when the cartridge is inserted."
+		(at 170.23 67.47 0)
 		(layer "Cmts.User")
 		(effects

Commit message: deep revision hardw & github info
Parts:
- moved R2 7.70 mm to (149.3, 90.2)
- moved D2 7.42 mm to (153.4, 87.1)
- moved D1 7.42 mm to (153.4, 94.5)
- moved R1 5.82 mm to (149.1, 98.0), turned to 0 degrees
- moved C1 0.38 mm to (137.9, 89.8)
- moved SW3 0.10 mm to (152.9, 104.5)
- moved SCR1 0.05 mm to (136.8, 86.0)
Routing:
- net /UI_BTN_SELECT: track 45.5 -> 42.9 mm, vias 0 -> 2
- net /UI_LD_READ: track 49.6 -> 47.0 mm
- net GND: track 22.8 -> 20.9 mm, vias 15 -> 45
- net /UI_BTN_BACK: track 48.4 -> 46.6 mm
- net /UI_SD_MOSI: track 30.1 -> 31.3 mm
- net /UI_BTN_NEXT: track 44.7 -> 43.7 mm
- net /UI_LD_WRITE: track 48.1 -> 47.5 mm
Other:
- board size 33.9 x 37.5 mm -> 30.8 x 36 mm
- board text added: "Pin#14 on back side is UI_Detect that close the ground laze when the cartridge is inserted."
- board text added: "Redesigned by Popopo (2026) Original design by Dr. Gusman"
- board text added: "Rereference original Cartridge for retro-compability and symbolic representation"
- board text added: "Ver 1.5a.L"
- board text added: "Ver 1.5a.S"
- board text added: "WayWayWay"
- board text removed: "2023 Redesigned by Popopo Original design by Dr. Gusman"
- board text removed: "Pin#14 is UI_Detect that close the ground laze when the cartridge is inserted."
- board text removed: "Ver 1.4e.L"

Commit message: upgrading last changes
Parts:
- moved D1 7.44 mm to (153.4, 87.1)
- moved D2 7.43 mm to (153.4, 94.5)
- moved R2 7.00 mm to (149.3, 97.2)
- moved R1 4.93 mm to (149.3, 93.1), turned to 90 degrees
Routing:
- net /UI_LD_READ: track 47.0 -> 52.1 mm
- net /UI_LD_WRITE: track 47.5 -> 45.7 mm
- net Net-(D1-A): track 3.91 -> 5.17 mm
- net GND: vias 45 -> 44
